File: design/UIRRC/uirrc.sch (EAGLE design)
At the start: 46 parts, among them IC1 TSOP38438, IC2 FT232RL, J1 UJ2-MIBH-G-SMT-TR, U1 ESP32-WROOM-32E_(16MB)

Commit message: Fixes #5
Parts:
- added C5: 1.0uF, rcl:C-EUC1206
- added IC3: MIC5205-3.3YM5-TR, MIC5205-3.3YM5-TR:MIC5205-3.3YM5-TR
- added S13: AYZ0102AGRLC, AYZ0102AGRLC:AYZ0102AGRLC
- added U2: 2479, 2479:2479
- R10, R11, R2, R3, R4: value 470 -> 471
Connections:
- new net N$11: S13.3, U2.+
- new net N$16: IC3.EN, IC3.IN, S13.2
- net +3V3: now also C5.1, IC3.OUT
- net GND: now also C5.2, IC3.GND, S13.1, U2.-
Other:
- note added: "Power Circuit"
Changed lines of the file:
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@@
 <part name="+3V5" library="supply1" library_urn="urn:adsk.eagle:library:371" deviceset="+3V3" device=""/>
 <part name="GND6" library="supply1" library_urn="urn:adsk.eagle:library:371" deviceset="GND" device=""/>
-<part name="R10" library="rcl" library_urn="urn:adsk.eagle:library:334" deviceset="R-EU_" device="R1206" package3d_urn="urn:adsk.eagle:package:23540/2" value="470"/>
+<part name="R10" library="rcl" library_urn="urn:adsk.eagle:library:334" deviceset="R-EU_" device="R1206" package3d_urn="urn:adsk.eagle:package:23540/2" value="471"/>
 <part name="LED5" library="led" library_urn="urn:adsk.eagle:library:259" deviceset="LED" device="CHIPLED_1206" package3d_urn="urn:adsk.eagle:package:15823/2"/>
 <part name="GND7" library="supply1" library_urn="urn:adsk.eagle:library:371" deviceset="GND" device=""/>
-<part name="R11" library="rcl" library_urn="urn:adsk.eagle:library:334" deviceset="R-EU_" device="R1206" package3d_urn="urn:adsk.eagle:package:23540/2" value="470"/>
+<part name="R11" library="rcl" library_urn="urn:adsk.eagle:library:334" deviceset="R-EU_" device="R1206" package3d_urn="urn:adsk.eagle:package:23540/2" value="471"/>
 <part name="LED6" library="led" library_urn="urn:adsk.eagle:library:259" deviceset="LED" device="CHIPLED_1206" package3d_urn="urn:adsk.eagle:package:15823/2"/>
 <part name="S3" library="EVP-BV2C3L000" deviceset="EVP-BV2C3L000" device=""/>
@@
 <part name="S2" library="AYZ0102AGRLC" deviceset="AYZ0102AGRLC" device=""/>
 <part name="LED2" library="CLVBA-FKA-CAEDH8BBB7A363" deviceset="CLVBA-FKA-CAEDH8BBB7A363" device=""/>
-<part name="R2" library="rcl" library_urn="urn:adsk.eagle:library:334" deviceset="R-EU_" device="R1206" package3d_urn="urn:adsk.eagle:package:23540/2" value="470"/>
-<part name="R3" library="rcl" library_urn="urn:adsk.eagle:library:334" deviceset="R-EU_" device="R1206" package3d_urn="urn:adsk.eagle:package:23540/2" value="470"/>
-<part name="R4" library="rcl" library_urn="urn:adsk.eagle:library:334" deviceset="R-EU_" device="R1206" package3d_urn="urn:adsk.eagle:package:23540/2" value="470"/>
+<part name="R2" library="rcl" library_urn="urn:adsk.eagle:library:334" deviceset="R-EU_" device="R1206" package3d_urn="urn:adsk.eagle:package:23540/2" value="471"/>
+<part name="R3" library="rcl" library_urn="urn:adsk.eagle:library:334" deviceset="R-EU_" device="R1206" package3d_urn="urn:adsk.eagle:package:23540/2" value="471"/>
+<part name="R4" library="rcl" library_urn="urn:adsk.eagle:library:334" deviceset="R-EU_" device="R1206" package3d_urn="urn:adsk.eagle:package:23540/2" value="471"/>
+<part name="U2" library="2479" deviceset="2479" device=""/>
+<part name="IC3" library="MIC5205-3.3YM5-TR" deviceset="MIC5205-3.3YM5-TR" device=""/>
+<part name="S13" library="AYZ0102AGRLC" deviceset="AYZ0102AGRLC" device=""/>
+<part name="+3V4" library="supply1" library_urn="urn:adsk.eagle:library:371" deviceset="+3V3" device=""/>
+<part name="GND4" library="supply1" library_urn="urn:adsk.eagle:library:371" deviceset="GND" device=""/>
+<part name="C5" library="rcl" library_urn="urn:adsk.eagle:library:334" deviceset="C-EU" device="C1206" package3d_urn="urn:adsk.eagle:package:23618/2" value="1.0uF"/>
+<part name="GND5" library="supply1" library_urn="urn:adsk.eagle:library:371" deviceset="GND" device=""/>
 </parts>
 <sheets>
@@
 <wire x1="22.86" y1="50.8" x2="22.86" y2="195.58" width="0.1524" layer="97"/>
 <text x="22.86" y="198.12" size="2.54" layer="97">Buttons</text>
+<wire x1="152.4" y1="233.68" x2="152.4" y2="187.96" width="0.1524" layer="97"/>
+<wire x1="152.4" y1="187.96" x2="246.38" y2="187.96" width="0.1524" layer="97"/>
+<wire x1="246.38" y1="187.96" x2="246.38" y2="233.68" width="0.1524" layer="97"/>
+<wire x1="246.38" y1="233.68" x2="152.4" y2="233.68" width="0.1524" layer="97"/>
+<text x="152.4" y="236.22" size="2.54" layer="97">Power Circuit</text>
 </plain>
 <instances>
@@
 <attribute name="NAME" x="186.69" y="105.6386" size="1.778" layer="95"/>
 <attribute name="VALUE" x="186.69" y="95.758" size="1.778" layer="96"/>
+</instance>
+<instance part="U2" gate="G$1" x="154.94" y="205.74" smashed="yes" rot="MR180">
+<attribute name="NAME" x="161.29" y="213.36" size="1.778" layer="95" rot="MR180" align="center-left"/>
+<attribute name="VALUE" x="161.29" y="215.9" size="1.778" layer="96" rot="MR180" align="center-left"/>
+</instance>
+<instance part="IC3" gate="G$1" x="198.12" y="208.28" smashed="yes">
+<attribute name="NAME" x="201.93" y="215.9" size="1.778" layer="95" align="center-left"/>
+<attribute name="VALUE" x="201.93" y="213.36" size="1.778" layer="96" align="center-left"/>
+</instance>
+<instance part="S13" gate="G$1" x="190.5" y="231.14" smashed="yes" rot="R270">
+<attribute name="NAME" x="162.56" y="229.87" size="1.778" layer="95" align="center-left"/>
+<attribute name="VALUE" x="162.56" y="227.33" size="1.778" layer="96" align="center-left"/>
+</instance>
+<instance part="+3V4" gate="G$1" x="236.22" y="210.82" smashed="yes">
+<attribute name="VALUE" x="238.76" y="215.9" size="1.778" layer="96" rot="R180"/>
+</instance>
+<instance part="GND4" gate="1" x="231.14" y="193.04" smashed="yes">
+<attribute name="VALUE" x="228.6" y="190.5" size="1.778" layer="96"/>
+</instance>
+<instance part="C5" gate="G$1" x="231.14" y="200.66" smashed="yes">
+<attribute name="NAME" x="232.664" y="201.041" size="1.778" layer="95"/>
+<attribute name="VALUE" x="232.664" y="195.961" size="1.778" layer="96"/>
+</instance>
+<instance part="GND5" gate="1" x="185.42" y="193.04" smashed="yes">
+<attribute name="VALUE" x="182.88" y="190.5" size="1.778" layer="96"/>
 </instance>
 </instances>
@@
 <wire x1="-26.67" y1="218.44" x2="-26.67" y2="217.17" width="0.1524" layer="91"/>
 </segment>
+<segment>
+<pinref part="GND4" gate="1" pin="GND"/>
+<pinref part="C5" gate="G$1" pin="2"/>
+</segment>
+<segment>
+<pinref part="U2" gate="G$1" pin="-"/>
+<wire x1="175.26" y1="205.74" x2="185.42" y2="205.74" width="0.1524" layer="91"/>
+<pinref part="S13" gate="G$1" pin="1"/>
+<wire x1="185.42" y1="205.74" x2="190.5" y2="205.74" width="0.1524" layer="91"/>
+<wire x1="190.5" y1="205.74" x2="190.5" y2="210.82" width="0.1524" layer="91"/>
+<pinref part="IC3" gate="G$1" pin="GND"/>
+<wire x1="198.12" y1="205.74" x2="190.5" y2="205.74" width="0.1524" layer="91"/>
+<junction x="190.5" y="205.74"/>
+<pinref part="GND5" gate="1" pin="GND"/>
+<wire x1="185.42" y1="195.58" x2="185.42" y2="205.74" width="0.1524" layer="91"/>
+<junction x="185.42" y="205.74"/>
+</segment>
 </net>
 <net name="+3V3" class="0">
@@
 <wire x1="-59.69" y1="209.55" x2="-48.26" y2="209.55" width="0.1524" layer="91"/>
 <wire x1="-48.26" y1="209.55" x2="-48.26" y2="210.82" width="0.1524" layer="91"/>
+</segment>
+<segment>
+<pinref part="IC3" gate="G$1" pin="OUT"/>
+<pinref part="+3V4" gate="G$1" pin="+3V3"/>
+<wire x1="223.52" y1="205.74" x2="231.14" y2="205.74" width="0.1524" layer="91"/>
+<wire x1="231.14" y1="205.74" x2="236.22" y2="205.74" width="0.1524" layer="91"/>
+<wire x1="236.22" y1="205.74" x2="236.22" y2="208.28" width="0.1524" layer="91"/>
+<pinref part="C5" gate="G$1" pin="1"/>
+<wire x1="231.14" y1="203.2" x2="231.14" y2="205.74" width="0.1524" layer="91"/>
+<junction x="231.14" y="205.74"/>
 </segment>
 </net>
@@
 </segment>
 </net>
+<net name="N$11" class="0">
+<segment>
+<pinref part="U2" gate="G$1" pin="+"/>
+<wire x1="175.26" y1="208.28" x2="185.42" y2="208.28" width="0.1524" layer="91"/>
+<pinref part="S13" gate="G$1" pin="3"/>
+<wire x1="185.42" y1="208.28" x2="185.42" y2="210.82" width="0.1524" layer="91"/>
+</segment>
+</net>
+<net name="N$16" class="0">
+<segment>
+<pinref part="S13" gate="G$1" pin="2"/>
+<wire x1="187.96" y1="210.82" x2="187.96" y2="208.28" width="0.1524" layer="91"/>
+<wire x1="187.96" y1="208.28" x2="198.12" y2="208.28" width="0.1524" layer="91"/>
+<pinref part="IC3" gate="G$1" pin="IN"/>
+<pinref part="IC3" gate="G$1" pin="EN"/>
+<wire x1="187.96" y1="208.28" x2="187.96" y2="203.2" width="0.1524" layer="91"/>
+<wire x1="187.96" y1="203.2" x2="198.12" y2="203.2" width="0.1524" layer="91"/>
+<junction x="187.96" y="208.28"/>
+</segment>
+</net>

Commit message: UART Programmer offboarded
Parts:
- removed C1, C2: 100nF, rcl:C-USC0402
- removed C3: 10nF, rcl:CPOL-USA
- removed C4: 4.7uF, rcl:CPOL-USD
- removed IC2: FT232RL, ftdichip:FT232RL
- removed J1: UJ2-MIBH-G-SMT-TR, UJ2-MIBH-G-SMT-TR:UJ2-MIBH-G-SMT-TR
- removed L1: Ferrite Bead, inductors:BLM15HB121SN1
- removed R5, R6: (no value), rcl:R-EU_R1206
- removed T2, T3: (no value), transistor:MMBT3904LT1-NPN-SOT23-BEC
- added JP1: (no value), pinhead:PINHD-1X4
Connections:
- removed net N$10: R5.2, T2.B
- removed net N$12: R6.2, T3.B
- removed net N$5: C3.+, J1.1, L1.1
- removed net N$6: IC2.USBDP, J1.3
- removed net N$7: IC2.USBDM, J1.2
- removed net N$8: C2.1, IC2.3V3OUT
- removed net USB_DTR: IC2.!DTR, R5.1, T3.C
- removed net USB_RTS: IC2.!RTS, R6.1, T2.E
- removed net VCC: C1.1, C4.+, IC2.VCC, IC2.VCCIO, L1.2
- net +3V3: now also JP1.1
- net EN: no longer T2.C
- net GND: now also JP1.2; no longer C1.2, C2.2, C3.-, C4.-, IC2.GND, IC2.GND@1, IC2.GND@2, IC2.GND@A, J1.5
- net IO0: no longer T3.E
- net USB_RXD: now also JP1.3; no longer IC2.RXD
- net USB_TXD: now also JP1.4; no longer IC2.TXD
Other:
- note removed: "RESET Handshakes"

Commit message: Fixes #10
Parts:
- removed C5: 1.0uF, rcl:C-EUC1206
- removed IC3: MIC5205-3.3YM5-TR, MIC5205-3.3YM5-TR:MIC5205-3.3YM5-TR
- removed LED6: (no value), led:LEDCHIPLED_1206
- removed R10, R11: 471, rcl:R-EU_R1206
- removed R12, R13, R14, R15, R16, R17, R18, R19, R20, R21: 1k, rcl:R-EU_R1206
- removed S10, S11, S12, S4, S5, S6, S7, S8, S9: EVP-BV2C3L000, EVP-BV2C3L000:EVP-BV2C3L000
- removed S13: AYZ0102AGRLC, AYZ0102AGRLC:AYZ0102AGRLC
- added C1: 1.0uF, rcl:C-EUC1206
- added IC2: MIC5205-3.3YM5-TR, MIC5205-3.3YM5-TR:MIC5205-3.3YM5-TR
- added LED4: CLVBA-FKA-CAEDH8BBB7A363, CLVBA-FKA-CAEDH8BBB7A363:CLVBA-FKA-CAEDH8BBB7A363
- added R5, R6: 471, rcl:R-EU_R1206
- added SW1, SW2, SW3, SW4, SW5, SW6, SW7, SW8, SW9: OMRON_B3SN-3112POMRON_B3SN-3112P_0_0, Omron - B3SN-3112P:OMRON_B3SN-3112POMRON_B3SN-3112P_0_0
- LED2: value CLVBA-FKA-CAEDH8BBB7A363 -> (none); device CLVBA-FKA-CAEDH8BBB7A363:CLVBA-FKA-CAEDH8BBB7A363 -> led:LEDCHIPLED_1206
- S3: value EVP-BV2C3L000 -> AYZ0102AGRLC; device EVP-BV2C3L000:EVP-BV2C3L000 -> AYZ0102AGRLC:AYZ0102AGRLC
- U1: value ESP32-WROOM-32E_(16MB) -> 2479; device ESP32-WROOM-32E__16MB_:ESP32-WROOM-32E_(16MB) -> 2479:2479
- U2: value 2479 -> ESP32-WROOM-32E_(16MB); device 2479:2479 -> ESP32-WROOM-32E__16MB_:ESP32-WROOM-32E_(16MB)
- renumbered LED5 to LED3
Connections:
- removed net BUTTON1: R13.1, S4.NO_2, U1.IO5
- removed net BUTTON2: R14.1, S5.NO_2, U1.IO2
- removed net BUTTON3: R15.1, S6.NO_2, U1.IO15
- removed net BUTTON4: R16.1, S7.NO_2, U1.IO13
- removed net BUTTON5: R17.1, S8.NO_2, U1.IO12
- removed net BUTTON6: R18.1, S9.NO_2, U1.IO14
- removed net BUTTON7: R19.1, S10.NO_2, U1.IO27
- removed net BUTTON8: R20.1, S11.NO_2, U1.IO33
- removed net BUTTON9: R21.1, S12.NO_2, U1.IO32
- new net BUTTON_C1: SW1.3, SW2.3, SW3.3, U2.IO13
- new net BUTTON_C2: SW4.3, SW5.3, SW6.3, U2.IO12
- new net BUTTON_C3: SW7.3, SW8.3, SW9.3, U2.IO14
- new net BUTTON_R1: SW1.1, SW4.1, SW7.1, U2.IO5
- new net BUTTON_R2: SW2.1, SW5.1, SW8.1, U2.IO2
- new net BUTTON_R3: SW3.1, SW6.1, SW9.1, U2.IO15
- net +3V3: now also C1.1, IC2.OUT, LED4.COMMON_ANODE, S3.3, U2.3V3; no longer C5.1, IC3.OUT, LED2.COMMON_ANODE, S1.3, S10.NO_1, S11.NO_1, S12.NO_1, S3.NO_1, S4.NO_1, S5.NO_1, S6.NO_1, S7.NO_1, S8.NO_1, S9.NO_1, U1.3V3
- net EN: now also U2.EN; no longer U1.EN
- net GND: now also C1.2, IC2.GND, R2.2, R3.2, S3.1, U1.-, U2.GND; no longer C5.2, IC3.GND, R10.2, R11.2, R12.2, R13.2, R14.2, R15.2, R16.2, R17.2, R18.2, R19.2, R20.2, R21.2, S13.1, U1.GND, U2.-
- net IO0: now also U2.IO0; no longer U1.IO0
- net IR_RX: now also U2.IO4; no longer U1.IO4
- net IR_TX: now also U2.IO25; no longer U1.IO25
- net LEARN_EN: now also S3.2, U2.IO35; no longer S1.2, U1.IO35
- net LEARN_LED: now also U2.IO18; no longer U1.IO18
- net N$11: now also S1.3, U1.+; no longer S13.3, U2.+
- net N$13: now also R4.1, U2.IO21; no longer R2.1, U1.IO21
- net N$14: now also R5.1, U2.IO22; no longer R3.1, U1.IO22
- net N$15: now also R6.1, U2.IO23; no longer R4.1, U1.IO23
- net N$16: now also IC2.EN, IC2.IN, S1.2; no longer IC3.EN, IC3.IN, S13.2
- net N$18: now also R3.1; no longer R10.1
- net N$20: now also LED2.C, R2.1; no longer LED6.C, R11.1
- net N$3: now also LED4.GREEN_(CATHODE), R4.2; no longer LED2.GREEN_(CATHODE), R2.2
- net N$4: now also LED4.BLUE_(CATHODE), R5.2; no longer LED2.BLUE_(CATHODE), R3.2
- net N$9: now also LED4.RED_(CATHODE), R6.2; no longer LED2.RED_(CATHODE), R4.2
- net PROFILE_T: now also U2.IO19; no longer R12.1, S3.NO_2, U1.IO19
- net USB_RXD: now also U2.TXD0; no longer U1.TXD0
- net USB_TXD: now also U2.RXD0; no longer U1.RXD0
- net WIFI_EN: now also U2.IO34; no longer U1.IO34
- net WIFI_LED: now also LED2.A, U2.IO17; no longer LED6.A, U1.IO17
Other:
- note added: "Button Matrix"
- note added: "UART Programmer Circuit"
- note removed: "Buttons"
- note removed: "USB to MCU UART Circuit"
- moved on the sheet: JP1, R2, R3, R4, S1
