File: design/UIRRC/uirrc.sch (EAGLE design)
At the start: 29 parts, among them IC1 TSOP38438, IC2 MIC5205-3.3YM5-TR, SW1 OMRON_B3SN-3112POMRON_B3SN-31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, SW2 OMRON_B3SN-3112POMRON_B3SN-31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, SW3 OMRON_B3SN-3112POMRON_B3SN-31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, SW4 OMRON_B3SN-3112POMRON_B3SN-31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, SW5 OMRON_B3SN-3112POMRON_B3SN-31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, SW6 OMRON_B3SN-3112POMRON_B3SN-31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, SW7 OMRON_B3SN-3112POMRON_B3SN-31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, SW8 OMRON_B3SN-3112POMRON_B3SN-31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

Commit message: Updated board design
Connections:
- net BUTTON_C1: now also SW1.1, SW4.1, SW7.1, U2.IO13; no longer SW1.3, SW2.3, SW3.3, U2.IO2
- net BUTTON_C2: now also SW2.1, SW5.1, SW8.1; no longer SW4.3, SW5.3, SW6.3
- net BUTTON_C3: now also SW3.1, SW6.1, SW9.1, U2.IO2; no longer SW7.3, SW8.3, SW9.3, U2.IO13
- net BUTTON_R1: now also SW1.3, SW2.3, SW3.3, U2.IO12; no longer SW1.1, SW4.1, SW7.1, U2.IO27
- net BUTTON_R2: now also SW4.3, SW5.3, SW6.3; no longer SW2.1, SW5.1, SW8.1
- net BUTTON_R3: now also SW7.3, SW8.3, SW9.3, U2.IO27; no longer SW3.1, SW6.1, SW9.1, U2.IO12
