File: design/UIRRC/uirrc.brd (EAGLE design)
At the start: 51.7 x 83.8 mm, 29 parts, among them IC1 TSOP38438, IC2 MIC5205-3.3YM5-TR, SW1 OMRON_B3SN-3112POMRON_B3SN-31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, SW2 OMRON_B3SN-3112POMRON_B3SN-31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, SW3 OMRON_B3SN-3112POMRON_B3SN-31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, SW4 OMRON_B3SN-3112POMRON_B3SN-31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, SW5 OMRON_B3SN-3112POMRON_B3SN-31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, SW6 OMRON_B3SN-3112POMRON_B3SN-31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, SW7 OMRON_B3SN-3112POMRON_B3SN-31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, SW8 OMRON_B3SN-3112POMRON_B3SN-31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

Commit message: Fixes #12
Parts:
- moved JP1 44.6 mm to (38.1, 43.8), flipped to the top, turned to 180 degrees
- moved SW7 42.0 mm to (8.89, 9.53)
- moved SW3 40.4 mm to (39.4, 36.8)
- moved LED4 35.6 mm to (5.08, 75.6), turned to 180 degrees
- moved R4 30.8 mm to (2.54, 69.2), turned to 90 degrees
- moved R5 30.2 mm to (3.81, 63.5), turned to 90 degrees
- moved R6 30.0 mm to (5.08, 57.8), turned to 90 degrees
- moved SW8 22.2 mm to (24.1, 9.53)
- moved SW4 21.8 mm to (8.89, 22.9)
- moved SW2 19.8 mm to (24.1, 36.8)
- moved SW6 18.9 mm to (39.4, 22.9)
- moved T1 16.3 mm to (29.2, 67.9), flipped to the bottom
- moved S2 12.9 mm to (45.1, 64.1)
- moved S3 11.7 mm to (45.1, 54.0)
- moved R1 11.3 mm to (22.9, 73.0), flipped to the bottom, turned to 270 degrees
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Connections:
- removed net EN: U2.3
- removed net PROFILE_T: U2.31
- net +3V3: now also U2.3
- net BUTTON_C1: now also U2.24; no longer U2.16
- net BUTTON_C2: now also U2.23; no longer U2.14
- net BUTTON_C3: now also U2.16; no longer U2.13
- net BUTTON_R1: now also U2.12; no longer U2.29
- net BUTTON_R2: now also U2.13; no longer U2.24
- net BUTTON_R3: now also U2.14; no longer U2.23
- net IR_RX: now also U2.6; no longer U2.26
- net IR_TX: now also U2.37; no longer U2.10
- net LEARN_EN: now also U2.31; no longer U2.7
- net N$13: now also U2.11; no longer U2.33
- net N$14: now also U2.10; no longer U2.36
- net N$15: now also U2.9; no longer U2.37
- net WIFI_EN: now also U2.33; no longer U2.6
- net WIFI_LED: now also U2.36; no longer U2.28
Routing:
- net GND: track 217.1 -> 8.69 mm, vias 0 -> 1
- net LEARN_EN: track 51.3 -> 16.5 mm
- net BUTTON_R2: track 97.3 -> 69.4 mm
- net LEARN_LED: track 29.6 -> 6.08 mm
- net WIFI_EN: track 44.1 -> 20.7 mm
- net IR_TX: track 26.1 -> 7.51 mm, vias 0 -> 1
- net N$1: track 20.8 -> 3.66 mm
- net N$11: track 59.8 -> 45.7 mm
- net WIFI_LED: track 19.1 -> 7.25 mm, vias 2 -> 0
- net BUTTON_C1: track 43.8 -> 55.0 mm, vias 4 -> 0
- net BUTTON_C2: track 60.0 -> 71.0 mm, vias 4 -> 0
- net USB_TXD: track 31.2 -> 22.6 mm
- net BUTTON_R1: track 62.7 -> 57.0 mm
- net N$16: track 7.27 -> 12.2 mm
- net N$13: track 18.5 -> 23.3 mm, vias 2 -> 0
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- added copper zone on layer 1, net GND
- added copper zone on layer 16, net GND
Other:
- board size 51.7 x 83.8 mm -> 47.9 x 80 mm
- board text added: "IR REMOTE | MUBARIZ & HADI"

Commit message: Updated board design
Parts:
- moved R1 6.38 mm to (29.2, 72.4), flipped to the top, turned to 0 degrees
- moved LED1 2.54 mm to (22.9, 75.6)
- moved T1 1.90 mm to (31.1, 67.9), flipped to the top
- moved IC2 1.42 mm to (36.2, 72.4), flipped to the top, turned to 180 degrees
- moved C1 0.64 mm to (35.6, 77.5), flipped to the top, turned to 0 degrees
- flipped S1 to the top, turned to 90 degrees
Connections:
- net BUTTON_C1: now also SW1.1, SW4.1, SW7.1, U2.16; no longer SW1.3, SW2.3, SW3.3, U2.24
- net BUTTON_C2: now also SW2.1, SW5.1, SW8.1; no longer SW4.3, SW5.3, SW6.3
- net BUTTON_C3: now also SW3.1, SW6.1, SW9.1, U2.24; no longer SW7.3, SW8.3, SW9.3, U2.16
- net BUTTON_R1: now also SW1.3, SW2.3, SW3.3, U2.14; no longer SW1.1, SW4.1, SW7.1, U2.12
- net BUTTON_R2: now also SW4.3, SW5.3, SW6.3; no longer SW2.1, SW5.1, SW8.1
- net BUTTON_R3: now also SW7.3, SW8.3, SW9.3, U2.12; no longer SW3.1, SW6.1, SW9.1, U2.14
Routing:
- net BUTTON_C2: track 71.0 -> 52.8 mm
- net BUTTON_C3: track 77.1 -> 65.6 mm
- net BUTTON_R2: track 69.4 -> 79.3 mm
- net BUTTON_R1: track 57.0 -> 66.0 mm, vias 4 -> 3
- net BUTTON_R3: track 83.3 -> 91.0 mm
- net +3V3: track 110.2 -> 117.6 mm, vias 1 -> 0
- net BUTTON_C1: track 55.0 -> 48.2 mm
- net N$11: track 45.7 -> 51.1 mm, vias 0 -> 1
- net N$2: track 7.88 -> 3.55 mm
- net USB_TXD: track 22.6 -> 18.6 mm
- net N$1: track 3.66 -> 7.36 mm
- net USB_RXD: track 24.2 -> 22.0 mm
- net WIFI_EN: track 20.7 -> 21.9 mm
- net GND: track 8.69 -> 7.53 mm, vias 1 -> 2
- net IR_TX: track 7.51 -> 7.24 mm, vias 1 -> 0
Other:
- board size 47.9 x 80 mm -> 47.9 x 80.6 mm

Commit message: add uml
Parts:
- moved R2 27.1 mm to (54.0, 80.6), turned to 90 degrees
- moved S1 27.0 mm to (62.9, 94.6)
- moved IC2 23.6 mm to (48.3, 92.7)
- moved S2 23.4 mm to (62.2, 80.0)
- moved JP1 22.4 mm to (58.4, 53.3)
- moved C1 21.7 mm to (43.2, 97.8)
- moved LED1 21.7 mm to (30.5, 95.9)
- moved R3 21.0 mm to (54.0, 61.0)
- moved R1 20.8 mm to (45.7, 85.1)
- moved IC1 20.8 mm to (20.3, 94.6)
- moved T1 20.4 mm to (47.6, 80.0)
- moved S3 20.3 mm to (62.2, 64.8)
- moved U2 19.9 mm to (28.6, 74.9)
- moved LED4 19.8 mm to (7.62, 95.2)
- moved LED3 19.3 mm to (48.3, 66.7)
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Routing:
- net BUTTON_R3: track 91.0 -> 128.2 mm
- net +3V3: track 117.6 -> 152.4 mm
- net BUTTON_C3: track 65.6 -> 98.7 mm
- net BUTTON_R2: track 79.3 -> 111.2 mm
- net BUTTON_C2: track 52.8 -> 84.2 mm
- net BUTTON_C1: track 48.2 -> 78.8 mm
- net N$11: track 51.1 -> 76.5 mm
- net BUTTON_R1: track 66.0 -> 87.5 mm
- net N$1: track 7.36 -> 19.8 mm
- net USB_TXD: track 18.6 -> 30.8 mm
- net USB_RXD: track 22.0 -> 33.8 mm
- net N$16: track 11.9 -> 21.8 mm
- net LEARN_EN: track 16.3 -> 25.6 mm
- net WIFI_EN: track 21.9 -> 29.4 mm
- net N$13: track 23.7 -> 30.9 mm
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Other:
- board size 47.9 x 80.6 mm -> 66.3 x 107.9 mm
